File: hardware/Connectors.kicad_sch (KiCad schematic)
At the start: 5 parts, among them J3 FTSH-107-01-L-D-K, J4 Conn_02x02_Counter_Clockwise

Commit message: changed out of stock parts
Parts:
- D10: Mouser Part Number 771-PESD5V0L2BT-T/R -> 771-PESD5V0S2BT-QR; Mouser Price/Stock https://www.mouser.pl/ProductDetail/Nexperia/PESD5V0L2BT215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 -> https://www.mouser.pl/pl/ProductDetail/Nexperia/PESD5V0S2BT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
- J3: Mouser Price/Stock https://www.mouser.co.uk/ProductDetail/Samtec/FTSH-107-01-L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 -> https://www.mouser.pl/en/ProductDetail/Semtech/UCLAMP3301D.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
- J4: Mouser  price/stock (none) -> https://www.mouser.pl/pl/ProductDetail/JST-Commercial/S4B-E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; Mouser part number (none) -> 306-S4B-EHLFSN
Changed lines of the file:
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@@
 			)
 		)
-		(property "Datasheet" ""
+		(property "Datasheet" "https://www.mouser.pl/datasheet/3/1070/1/eEH.pdf"
 			(at 152.4 50.8 0)
 			(hide yes)
@@
 		)
 		(property "Description" "Generic connector, double row, 02x02, counter clockwise pin numbering scheme (similar to DIP package numbering), script generated (kicad-library-utils/schlib/autogen/connector/)"
+			(at 152.4 50.8 0)
+			(hide yes)
+			(show_name no)
+			(do_not_autoplace no)
+			(effects
+				(font
+					(size 1.27 1.27)
+				)
+			)
+		)
+		(property "Mouser part number" "306-S4B-EHLFSN"
+			(at 152.4 50.8 0)
+			(hide yes)
+			(show_name no)
+			(do_not_autoplace no)
+			(effects
+				(font
+					(size 1.27 1.27)
+				)
+			)
+		)
+		(property "Mouser  price/stock" "https://www.mouser.pl/pl/ProductDetail/JST-Commercial/S4B-EHLFSN?qs=QpmGXVUTftGwDl%2F7pWjViw%3D%3D"
 			(at 152.4 50.8 0)
 			(hide yes)
@@
 			)
 		)
-		(property "Datasheet" "https://assets.nexperia.com/documents/data-sheet/PESD5V0L2BT.pdf"
+		(property "Datasheet" "https://assets.nexperia.com/documents/data-sheet/PESD5V0S2BT-Q.pdf"
 			(at 110.49 50.8 0)
 			(hide yes)
@@
 			)
 		)
-		(property "Description" "Bidirectional dual transient-voltage-suppression diode, center on pin 3"
+		(property "Description" "ESD Protection Diodes / TVS Diodes PESD5V0S2BT-Q/SOT23/TO-236AB"
 			(at 114.3 50.8 0)
 			(hide yes)
@@
 			)
 		)
-		(property "Mouser Part Number" "771-PESD5V0L2BT-T/R"
+		(property "Mouser Part Number" "771-PESD5V0S2BT-QR"
 			(at 114.3 50.8 0)
 			(hide yes)
@@
 			)
 		)
-		(property "Mouser Price/Stock" "https://www.mouser.pl/ProductDetail/Nexperia/PESD5V0L2BT215?qs=LOCUfHb8d9sw%2B%2FcZzpNtzw%3D%3D"
+		(property "Mouser Price/Stock" "https://www.mouser.pl/pl/ProductDetail/Nexperia/PESD5V0S2BT-QR?qs=3Rah4i%252BhyCEGtuWGhtDKxg%3D%3D"
 			(at 114.3 50.8 0)
 			(hide yes)
@@
 			)
 		)
-		(property "Mouser Price/Stock" "https://www.mouser.co.uk/ProductDetail/Samtec/FTSH-107-01-L-D-K?qs=%252BZP6%2F%252BtExtDf9U3LcTl7MA%3D%3D"
+		(property "Mouser Price/Stock" "https://www.mouser.pl/en/ProductDetail/Semtech/UCLAMP3301D.TCT?qs=rBWM4%252BvDhIcs1MIPFV0RMQ%3D%3D"
 			(at 179.07 696.52 0)
 			(hide yes)

Commit message: fixed mouser links
Parts:
- J3: Mouser Price/Stock https://www.mouser.pl/en/ProductDetail/Semtech/UCLAMP3301D.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 -> https://www.mouser.pl/pl/ProductDetail/Samtec/FTSH-107-01-L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
Changed lines of the file:
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@@
 			)
 		)
-		(property "Mouser Price/Stock" "https://www.mouser.pl/en/ProductDetail/Semtech/UCLAMP3301D.TCT?qs=rBWM4%252BvDhIcs1MIPFV0RMQ%3D%3D"
+		(property "Mouser Price/Stock" "https://www.mouser.pl/pl/ProductDetail/Samtec/FTSH-107-01-L-D-K?qs=%252BZP6%2F%252BtExtDf9U3LcTl7MA%3D%3D"
 			(at 179.07 696.52 0)
 			(hide yes)
